File: Quad_ESC_adapter.brd (EAGLE design)
At the start: 101.6 x 41.1 mm, 13 parts, among them J1 IBPD-SOCKET, J2 IBPD-SOCKET, J3 IBPD-SOCKET, J4 IBPD-SOCKET

Commit message: check this
Parts:
- removed U$1: LUMENIER_QUAD, AUX, Lumenier ESC:LUMENIER_QUAD
- added U$10: LUMENIER_QUAD-NO-CUT, Lumenier ESC:LUMENIER_QUAD-NO-CUT
- moved H3 114.8 mm to (-14.5, 17.3), flipped to the bottom
- moved C1 81.9 mm to (-14.5, -33.8), flipped to the top, turned to 0 degrees
- moved H2 79.9 mm to (80.5, 37.8), flipped to the bottom
- moved C6 78.6 mm to (-14.5, -22.5), flipped to the top
- moved J4 18.0 mm to (73.4, 6.99)
- moved J3 17.8 mm to (73.5, 27.6)
- moved H1 17.8 mm to (-14.5, 37.9), flipped to the bottom
- moved U$2 17.8 mm to (-17.8, 0.00)
- moved H4 17.7 mm to (80.5, 17.3), flipped to the bottom
- moved J1 17.7 mm to (-7.37, 27.6)
- moved J2 17.6 mm to (-7.37, 6.99)
- moved C5 16.5 mm to (28.8, 9.27), turned to 90 degrees
Connections:
- net 12V: now also U$10.VIN; no longer U$1.VIN
- net ESC1_B: now also U$10.1; no longer U$1.1
- net ESC1_R: now also U$10.3; no longer U$1.3
- net ESC1_Y: now also U$10.2; no longer U$1.2
- net ESC2_B: now also U$10.4; no longer U$1.4
- net ESC2_R: now also U$10.6; no longer U$1.6
- net ESC2_Y: now also U$10.5; no longer U$1.5
- net ESC3_B: now also U$10.12; no longer U$1.12
- net ESC3_R: now also U$10.10; no longer U$1.10
- net ESC3_Y: now also U$10.11; no longer U$1.11
- net ESC4_B: now also U$10.9; no longer U$1.9
- net ESC4_R: now also U$10.7; no longer U$1.7
- net ESC4_Y: now also U$10.8; no longer U$1.8
- net GND: now also U$10.GND; no longer U$1.GND
Routing:
- added copper zone on layer 16, net ESC1_B
- added copper zone on layer 16, net ESC1_R
- added copper zone on layer 16, net ESC1_Y
- added copper zone on layer 16, net ESC2_B
- added copper zone on layer 16, net ESC2_R
- added copper zone on layer 16, net ESC2_Y
- added copper zone on layer 16, net ESC3_B
- added copper zone on layer 16, net ESC3_R
- added copper zone on layer 16, net ESC3_Y
- added copper zone on layer 16, net ESC4_B
- added copper zone on layer 16, net ESC4_R
- added copper zone on layer 16, net ESC4_Y
Other:
- outline, holes or cut-outs redrawn
- board text added: "12V"
- board text added: "GND"

Commit message: check this
Changed lines of the file:
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@@
 <contactref element="C6" pad="-"/>
 <contactref element="C1" pad="-"/>
-<wire x1="29.464" y1="38.862" x2="32.004" y2="38.862" width="0" layer="19" extent="1-1"/>
-<wire x1="32.004" y1="36.322" x2="32.004" y2="38.862" width="0" layer="19" extent="1-1"/>
-<wire x1="29.464" y1="36.322" x2="29.464" y2="38.862" width="0" layer="19" extent="1-1"/>
-<wire x1="26.924" y1="38.862" x2="29.464" y2="38.862" width="0" layer="19" extent="1-1"/>
-<wire x1="26.924" y1="36.322" x2="29.464" y2="36.322" width="0" layer="19" extent="1-1"/>
-<wire x1="24.384" y1="38.862" x2="26.924" y2="38.862" width="0" layer="19" extent="1-1"/>
-<wire x1="21.844" y1="38.862" x2="24.384" y2="38.862" width="0" layer="19" extent="1-1"/>
-<wire x1="24.384" y1="36.322" x2="26.924" y2="36.322" width="0" layer="19" extent="1-1"/>
-<wire x1="19.304" y1="38.862" x2="21.844" y2="38.862" width="0" layer="19" extent="1-1"/>
-<wire x1="21.844" y1="36.322" x2="21.844" y2="38.862" width="0" layer="19" extent="1-1"/>
-<wire x1="19.304" y1="36.322" x2="19.304" y2="38.862" width="0" layer="19" extent="1-1"/>
-<wire x1="29.464" y1="33.528" x2="29.464" y2="36.322" width="0" layer="19" extent="1-1"/>
-<wire x1="28.543" y1="30.878" x2="29.464" y2="33.528" width="0" layer="19" extent="1-1"/>
-<wire x1="28.194" y1="28.194" x2="28.543" y2="30.878" width="0" layer="19" extent="1-1"/>
-<wire x1="26.162" y1="28.448" x2="28.194" y2="28.194" width="0" layer="19" extent="1-1"/>
-<wire x1="24.638" y1="29.718" x2="26.162" y2="28.448" width="0" layer="19" extent="1-1"/>
-<wire x1="24.638" y1="31.496" x2="24.638" y2="29.718" width="0" layer="19" extent="1-1"/>
-<wire x1="23.622" y1="33.02" x2="24.638" y2="31.496" width="0" layer="19" extent="1-1"/>
-<wire x1="22.606" y1="31.496" x2="23.622" y2="33.02" width="0" layer="19" extent="1-1"/>
-<wire x1="22.098" y1="29.718" x2="22.606" y2="31.496" width="0" layer="19" extent="1-1"/>
-<wire x1="23.114" y1="28.448" x2="22.098" y2="29.718" width="0" layer="19" extent="1-1"/>
-<wire x1="15.748" y1="39.116" x2="19.304" y2="38.862" width="0" layer="19" extent="1-1"/>
-<wire x1="15.748" y1="36.068" x2="15.748" y2="39.116" width="0" layer="19" extent="1-1"/>
-<wire x1="28.829" y1="13.471" x2="23.114" y2="28.448" width="0" layer="19" extent="1-1"/>
-<wire x1="-10.278" y1="-22.479" x2="28.829" y2="13.471" width="0" layer="19" extent="1-1"/>
-<wire x1="-10.278" y1="-33.782" x2="-10.278" y2="-22.479" width="0" layer="19" extent="1-1"/>
+<wire x1="-10.278" y1="-22.479" x2="-10.278" y2="-33.782" width="0" layer="19" extent="1-1"/>
+<wire x1="28.829" y1="13.471" x2="-10.278" y2="-22.479" width="0" layer="19" extent="1-16"/>
 </signal>
 <signal name="ESC4_B">
@@
 <vertex x="59.3344" y="16.764"/>
 <vertex x="86.106" y="16.764"/>
-<vertex x="86.106" y="9.906"/>
-<vertex x="59.3344" y="9.906"/>
+<vertex x="86.106" y="10.0584"/>
+<vertex x="59.3344" y="10.0584"/>
 </polygon>
 <polygon width="0.1524" layer="1" thermals="no">
@@
 <vertex x="59.3852" y="16.7894"/>
 <vertex x="86.868" y="16.7894"/>
-<vertex x="86.868" y="9.906"/>
-<vertex x="59.3852" y="9.906"/>
+<vertex x="86.868" y="10.0584"/>
+<vertex x="59.3852" y="10.0584"/>
 </polygon>
 <polygon width="0.1524" layer="16" thermals="no">
@@
 </polygon>
 <contactref element="J4" pad="1"/>
-<wire x1="56.033" y1="14.428" x2="69.6595" y2="11.176" width="0" layer="19" extent="1-1"/>
 </signal>
 <signal name="ESC4_Y">
@@
 <vertex x="73.279" y="5.08"/>
 </polygon>
-<wire x1="56.033" y1="8.858" x2="69.6595" y2="6.985" width="0" layer="19" extent="1-1"/>
 </signal>
 <signal name="ESC4_R">
@@
 </polygon>
 <contactref element="J4" pad="3"/>
-<wire x1="56.033" y1="3.288" x2="69.6595" y2="2.794" width="0" layer="19" extent="1-1"/>
 </signal>
 <signal name="ESC3_B">
@@
 </polygon>
 <contactref element="J3" pad="1"/>
-<wire x1="56.033" y1="31.128" x2="69.7865" y2="31.75" width="0" layer="19" extent="1-1"/>
 </signal>
 <signal name="ESC3_Y">
@@
 <vertex x="60.071" y="28.448"/>
 </polygon>
-<wire x1="56.033" y1="25.558" x2="69.7865" y2="27.559" width="0" layer="19" extent="1-1"/>
 </signal>
 <signal name="ESC3_R">
@@
 </polygon>
 <contactref element="J3" pad="3"/>
-<wire x1="56.033" y1="19.988" x2="69.7865" y2="23.368" width="0" layer="19" extent="1-1"/>
 </signal>
 <signal name="ESC2_B">
@@
 </polygon>
 <contactref element="J2" pad="3"/>
-<wire x1="-3.6195" y1="11.176" x2="10.033" y2="14.428" width="0" layer="19" extent="1-1"/>
 </signal>
 <signal name="ESC2_Y">
@@
 <vertex x="-7.239" y="5.461"/>
 </polygon>
-<wire x1="-3.6195" y1="6.985" x2="10.033" y2="8.858" width="0" layer="19" extent="1-1"/>
 </signal>
 <signal name="ESC2_R">
@@
 </polygon>
 <contactref element="J2" pad="1"/>
-<wire x1="-3.6195" y1="2.794" x2="10.033" y2="3.288" width="0" layer="19" extent="1-1"/>
 </signal>
 <signal name="ESC1_Y">
@@
 <vertex x="5.969" y="28.448"/>
 </polygon>
-<wire x1="-3.6195" y1="27.559" x2="10.033" y2="25.558" width="0" layer="19" extent="1-1"/>
 </signal>
 <signal name="ESC1_R">
@@
 </polygon>
 <contactref element="J1" pad="1"/>
-<wire x1="-3.6195" y1="23.368" x2="10.033" y2="19.988" width="0" layer="19" extent="1-1"/>
 </signal>
 <signal name="12V">
@@
 <via x="26.67" y="2.667" extent="1-16" drill="0.6"/>
 <via x="28.194" y="1.397" extent="1-16" drill="0.6" alwaysstop="yes"/>
-<via x="29.464" y="2.667" extent="1-16" drill="0.6"/>
+<via x="29.591" y="2.159" extent="1-16" drill="0.6"/>
 <via x="31.115" y="1.397" extent="1-16" drill="0.6" alwaysstop="yes"/>
 <via x="32.258" y="2.667" extent="1-16" drill="0.6"/>
@@
 <contactref element="C6" pad="+"/>
 <contactref element="C1" pad="+"/>
-<wire x1="50.165" y1="36.195" x2="50.165" y2="38.989" width="0" layer="19" extent="1-1"/>
-<wire x1="47.244" y1="38.862" x2="50.165" y2="38.989" width="0" layer="19" extent="1-1"/>
-<wire x1="44.704" y1="38.862" x2="47.244" y2="38.862" width="0" layer="19" extent="1-1"/>
-<wire x1="47.244" y1="36.322" x2="47.244" y2="38.862" width="0" layer="19" extent="1-1"/>
-<wire x1="42.164" y1="38.862" x2="44.704" y2="38.862" width="0" layer="19" extent="1-1"/>
-<wire x1="44.704" y1="36.322" x2="44.704" y2="38.862" width="0" layer="19" extent="1-1"/>
-<wire x1="42.164" y1="36.322" x2="42.164" y2="38.862" width="0" layer="19" extent="1-1"/>
-<wire x1="39.624" y1="38.862" x2="42.164" y2="38.862" width="0" layer="19" extent="1-1"/>
-<wire x1="37.084" y1="38.862" x2="39.624" y2="38.862" width="0" layer="19" extent="1-1"/>
-<wire x1="39.624" y1="36.322" x2="42.164" y2="36.322" width="0" layer="19" extent="1-1"/>
-<wire x1="37.084" y1="36.322" x2="37.084" y2="38.862" width="0" layer="19" extent="1-1"/>
-<wire x1="34.544" y1="38.862" x2="37.084" y2="38.862" width="0" layer="19" extent="1-1"/>
-<wire x1="34.544" y1="36.322" x2="37.084" y2="36.322" width="0" layer="19" extent="1-1"/>
-<wire x1="39.497" y1="33.655" x2="39.624" y2="36.322" width="0" layer="19" extent="1-1"/>
-<wire x1="41.021" y1="32.893" x2="39.497" y2="33.655" width="0" layer="19" extent="1-1"/>
-<wire x1="41.021" y1="31.369" x2="41.021" y2="32.893" width="0" layer="19" extent="1-1"/>
-<wire x1="37.465" y1="33.401" x2="39.497" y2="33.655" width="0" layer="19" extent="1-1"/>
-<wire x1="37.523" y1="30.878" x2="37.465" y2="33.401" width="0" layer="19" extent="1-1"/>
-<wire x1="43.561" y1="31.369" x2="41.021" y2="31.369" width="0" layer="19" extent="1-1"/>
-<wire x1="43.561" y1="32.893" x2="43.561" y2="31.369" width="0" layer="19" extent="1-1"/>
-<wire x1="34.925" y1="33.401" x2="37.465" y2="33.401" width="0" layer="19" extent="1-1"/>
-<wire x1="43.18" y1="5.715" x2="43.561" y2="31.369" width="0" layer="19" extent="1-1"/>
-<wire x1="41.529" y1="2.921" x2="43.18" y2="5.715" width="0" layer="19" extent="1-1"/>
-<wire x1="40.132" y1="1.397" x2="41.529" y2="2.921" width="0" layer="19" extent="1-1"/>
-<wire x1="38.608" y1="2.667" x2="40.132" y2="1.397" width="0" layer="19" extent="1-1"/>
-<wire x1="36.83" y1="1.397" x2="38.608" y2="2.667" width="0" layer="19" extent="1-1"/>
-<wire x1="35.306" y1="2.794" x2="36.83" y2="1.397" width="0" layer="19" extent="1-1"/>
-<wire x1="33.909" y1="1.397" x2="35.306" y2="2.794" width="0" layer="19" extent="1-1"/>
-<wire x1="32.258" y1="2.667" x2="33.909" y2="1.397" width="0" layer="19" extent="1-1"/>
-<wire x1="31.115" y1="1.397" x2="32.258" y2="2.667" width="0" layer="19" extent="1-1"/>
-<wire x1="29.464" y1="2.667" x2="31.115" y2="1.397" width="0" layer="19" extent="1-1"/>
-<wire x1="28.194" y1="1.397" x2="29.464" y2="2.667" width="0" layer="19" extent="1-1"/>
-<wire x1="26.67" y1="2.667" x2="28.194" y2="1.397" width="0" layer="19" extent="1-1"/>
-<wire x1="25.273" y1="1.397" x2="26.67" y2="2.667" width="0" layer="19" extent="1-1"/>
-<wire x1="23.749" y1="3.175" x2="25.273" y2="1.397" width="0" layer="19" extent="1-1"/>
-<wire x1="22.479" y1="5.461" x2="23.749" y2="3.175" width="0" layer="19" extent="1-1"/>
-<wire x1="28.829" y1="5.071" x2="22.479" y2="5.461" width="0" layer="19" extent="1-1"/>
-<wire x1="-18.678" y1="-22.479" x2="28.829" y2="5.071" width="0" layer="19" extent="1-1"/>
-<wire x1="-18.678" y1="-33.782" x2="-18.678" y2="-22.479" width="0" layer="19" extent="1-1"/>
+<wire x1="-18.678" y1="-22.479" x2="-18.678" y2="-33.782" width="0" layer="19" extent="1-1"/>
+<wire x1="23.749" y1="3.175" x2="-18.678" y2="-22.479" width="0" layer="19" extent="1-1"/>
 </signal>
 <signal name="ESC1_B">
@@
 </polygon>
 <contactref element="J1" pad="3"/>
-<wire x1="-3.6195" y1="31.75" x2="10.033" y2="31.128" width="0" layer="19" extent="1-1"/>
 </signal>
 </signals>
