File: Old Changes/Quad_ESC_controller.sch (EAGLE design)
At the start: 27 parts, among them IC1 OP-AMP, Y1 ECS-80-S-4X

Commit message: .
Parts:
- added J1, J10, J11, J2, J3, J6, J8: (no value), SparkFun-Connectors:CONN_01
- added OP-AMP, OP-AMP1: LM2904S, IC, LM2904:LM2904S
- J7: device SparkFun-Connectors:CONN_06SILK_FEMALE_PTH -> SparkFun-Connectors:CONN_01
Connections:
- net +3V3: now also OP-AMP1P.V+, OP-AMPP.V+
- net ADC: no longer J7.1
- net CAN_H: now also J10.1
- net CAN_L: now also J11.1
- net CAN_RX: now also J7.1
- net CAN_TX: now also J6.1
- net GND: now also OP-AMP1P.V-, OP-AMPP.V-
- net N$6: now also J8.1, OP-AMP1A.IN-; no longer IC1G1.-IN
- net NRST: now also J3.1
- net SWCLK: now also J1.1
- net SWDIO: now also J2.1
- net TIM3_CH1: no longer J7.3
- net TIM3_CH2: no longer J7.4
- net TIM3_CH3: no longer J7.5
- net TIM3_CH4: no longer J7.6
- net TLM: now also OP-AMP1A.OUT; no longer IC1G1.OUT
- net TLM_ESC: now also OP-AMP1A.IN+; no longer IC1G1.+IN, J7.2
Other:
- note added: "Not in stock, but still made"
- note removed: "ALL ONE OP-AMP - LM358"
- note removed: "Test points"
